File: overview.kicad_sch (KiCad schematic)
At the start: 2 parts, among them U1 SN74LVC8T245, U2 SN75160BDW

Commit message: Pre Ki10 migration
Other:
- sheet Microcontroller ports: added DIO[0..7]; removed none
Changed lines of the file:
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@@
+			)
+		)
+		(pin "DIO[0..7]" bidirectional
+			(at 152.4 104.14 0)
+			(effects
+				(font
+					(size 1.27 1.27)
+				)
+				(justify right)
 			)
 		)
