File: gpib_controller.kicad_pcb (KiCad board)
At the start: 4 copper layers, 55.1 x 55.1 mm, 44 parts, among them J1 112-024-113R001, J2 FTSH-105-01-L-DV-K, J3 RJHSE5380, J4 USB4085-GF-A, U1 SN74LVC8T245PWR, U2 SN74LVC07APWR, U3 STM32H533RETx, U4 PTS645SH43SMTR92 LFS, U5 THVD1451D, U6 SN74LVC1G07DCKR, U7 SN74LVC14APWR, U8 USBLC6-2SC6, U9 TPSM861253RDXR, Y1 MU00525-32.768K, Y2 CS10820-24M

Commit message: Final touches
Connections:
- U3 pad 20: /Overview/GPIB Transceiver/SRQ_SENSE -> unconnected-(U3H-PA4-Pad20)
- U3 pad 21: /Overview/GPIB Transceiver/DAV_SENSE -> unconnected-(U3G-PA5(SPI1_SCK)-Pad21)
- U3 pad 22: /Overview/GPIB Transceiver/NRFD_SENSE -> unconnected-(U3G-PA6(SPI1_MISO)-Pad22)
- U3 pad 23: /Overview/GPIB Transceiver/NDAC_SENSE -> /Overview/GPIB Transceiver/EOI_SENSE
- U3 pad 40: unconnected-(U3H-PC9-Pad40) -> /Overview/GPIB Transceiver/NRFD_SENSE
- U3 pad 41: unconnected-(U3H-PA8-Pad41) -> /Overview/GPIB Transceiver/DAV_SENSE
- U3 pad 42: unconnected-(U3H-PA9-Pad42) -> /Overview/GPIB Transceiver/SRQ_SENSE
- U3 pad 43: unconnected-(U3H-PA10-Pad43) -> /Overview/GPIB Transceiver/NDAC_SENSE
- U3 pad 50: /Overview/GPIB Transceiver/EOI_SENSE -> unconnected-(U3H-PA15(JTDI)-Pad50)
- U7 pad 3: /Overview/Connectors/EOI -> /Overview/Connectors/NDAC
- U7 pad 4: /Overview/GPIB Transceiver/EOI_SENSE -> /Overview/GPIB Transceiver/NDAC_SENSE
- U7 pad 5: /Overview/Connectors/NDAC -> /Overview/Connectors/EOI
- U7 pad 6: /Overview/GPIB Transceiver/NDAC_SENSE -> /Overview/GPIB Transceiver/EOI_SENSE
Routing:
- net /Overview/GPIB Transceiver/EOI_SENSE: track 0.00 -> 23.1 mm, vias 0 -> 2
- net /Overview/GPIB Transceiver/SRQ_SENSE: track 0.00 -> 20.9 mm
- net /Overview/GPIB Transceiver/NDAC_SENSE: track 0.00 -> 20.6 mm
- net /Overview/Connectors/DAV: track 35.0 -> 52.7 mm, vias 0 -> 1
- net /Overview/GPIB Transceiver/DAV_SENSE: track 0.00 -> 16.9 mm
- net /Overview/Connectors/NRFD: track 31.3 -> 47.3 mm, vias 0 -> 1
- net /Overview/GPIB Transceiver/NRFD_SENSE: track 0.00 -> 14.6 mm
- net +3V3: track 32.2 -> 42.3 mm, vias 3 -> 4
- net /Overview/Connectors/EOI: track 40.1 -> 49.8 mm
- net GND: track 91.6 -> 99.0 mm, vias 3 -> 5
- net /Overview/Connectors/NDAC: track 28.9 -> 34.4 mm
- net /Overview/Connectors/SRQ: track 14.2 -> 18.0 mm
- net +5V: track 64.9 -> 66.7 mm, vias 0 -> 1

Commit message: PCB finished, prior to rename and graphics
Parts:
- moved C10 19.8 mm to (145.1, 86.2), turned to 180 degrees
- moved U4 10.4 mm to (145.0, 92.0)
- moved J2 8.42 mm to (145.0, 102.4)
Routing:
- net +5V: track 66.7 -> 144.5 mm, vias 1 -> 2
- net GND: track 99.0 -> 149.5 mm, vias 5 -> 11
- net /Overview/Microcontroller/CTRL_RX: track 0.00 -> 36.3 mm, vias 0 -> 2
- net /Overview/Microcontroller/CTRL_TX: track 0.00 -> 36.1 mm, vias 0 -> 2
- net Net-(J2-NRST): track 12.9 -> 46.0 mm, vias 0 -> 2
- net /Overview/Microcontroller/iUSB_DM: track 0.00 -> 26.3 mm, vias 0 -> 2
- net /Overview/Microcontroller/iUSB_DP: track 0.00 -> 23.8 mm, vias 0 -> 2
- net /Overview/Microcontroller/VCAP: track 4.12 -> 17.7 mm
- net +3V3: track 42.3 -> 53.0 mm, vias 4 -> 9
- net Net-(J2-SWCLK): track 10.9 -> 17.8 mm
- net Net-(J2-SWDIO): track 5.58 -> 11.1 mm
- net /Overview/Connectors/CTRL_TX_N: track 23.4 -> 20.6 mm
- net /Overview/Connectors/CTRL_RX_N: track 18.5 -> 16.3 mm
- net /Overview/Connectors/CTRL_RX_P: track 10.1 -> 10.8 mm

Commit message: LINCs the name.
Routing:
- net GND: track 149.5 -> 130.6 mm, vias 11 -> 10
- added copper zone on F.Cu, net GND
Other:
- board size 55.1 x 55.1 mm -> 55.1 x 57.9 mm
- board text added: "ATN"
- board text added: "DAV"
- board text added: "DIO1"
- board text added: "DIO2"
- board text added: "DIO3"
- board text added: "DIO4"
- board text added: "DIO5"
- board text added: "DIO6"
- board text added: "DIO7"
- board text added: "DIO8"
- board text added: "EOI"
- board text added: "GND"
- board text added: "IFC"
- board text added: "NDAC"
- board text added: "NRFD"
- board text added: "REN"
- board text added: "SRQ"
- board text added: "U1"
